File: Hardware/PipeWatch/Photowiederstand.kicad_sch (KiCad schematic)
At the start: 3 parts

Commit message: Changed the scematic page Labeling
Other:
- company: (none) -> Felix Pelster
Changed lines of the file:
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@@
 	(generator_version "9.0")
 	(paper "A4")
+	(title_block
+		(date "2025-09-24")
+		(company "Felix Pelster")
+	)
 	(junction
 		(at 123.19 101.6)
