File: Hardware/PipeWatch/PipeWatch.kicad_sch (KiCad schematic)
At the start: 24 parts, among them J1 WJ126V-5.0-2P, U1 IRM-10-5_C20618064, U3 ESP32-S3-WROOM-1-N16R8, U5 XIAO-ESP32-S3-DIP

Commit message: Changed the scematic page Labeling
Other:
- company: (none) -> Felix Pelster
- title: (none) -> Pipe Watch
Changed lines of the file:
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@@
 	(generator_version "9.0")
 	(paper "A4")
+	(title_block
+		(title "Pipe Watch")
+		(date "2025-09-24")
+		(company "Felix Pelster")
+	)
 	(junction
 		(at 40.64 53.34)
