File: Hardware/PipeWatch/Taster.kicad_sch (KiCad schematic)
At the start: 4 parts, among them J3 Taster, J4 TasterLED

Commit message: Added Ten Sensor
Parts:
- removed J4: TasterLED, Connector_PinHeader_2.54mm:PinHeader_1x02_P2.54mm_Vertical, symbol Connector:Conn_01x02_Socket
Changed lines of the file:
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@@
-	)
-	(symbol
-		(lib_id "Connector:Conn_01x02_Socket")
-		(at 165.1 105.41 0)
-		(unit 1)
-		(exclude_from_sim no)
-		(in_bom yes)
-		(on_board yes)
-		(dnp no)
-		(fields_autoplaced yes)
-		(property "Reference" "J4"
-			(at 166.37 105.4099 0)
-			(effects
-				(font
-					(size 1.27 1.27)
-				)
-				(justify left)
-			)
-		)
-		(property "Value" "TasterLED"
-			(at 166.37 107.9499 0)
-			(effects
-				(font
-					(size 1.27 1.27)
-				)
-				(justify left)
-			)
-		)
-		(property "Footprint" "Connector_PinHeader_2.54mm:PinHeader_1x02_P2.54mm_Vertical"
-			(at 165.1 105.41 0)
-			(effects
-				(font
-					(size 1.27 1.27)
-				)
-				(hide yes)
-			)
-		)
-		(property "Datasheet" "~"
-			(at 165.1 105.41 0)
-			(effects
-				(font
-					(size 1.27 1.27)
-				)
-				(hide yes)
-			)
-		)
-		(property "Description" "Generic connector, single row, 01x02, script generated"
-			(at 165.1 105.41 0)
-			(effects
-				(font
-					(size 1.27 1.27)
-				)
-				(hide yes)
-			)
-		)
-		(pin "1"
-		)
-		(pin "2"
-		)
-		(instances
-			(project ""
-				(path "/149975cd-655c-40c3-be76-7a7ba16694c7/d82a02c7-ee87-4bf8-a44b-b037fa66d3cb"
-					(reference "J4")
-					(unit 1)
-				)
-			)
-		)
 	)
 	(symbol

Commit message: Changed the scematic page Labeling
Other:
- company: (none) -> Felix Pelster
Changed lines of the file:
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@@
 	(generator_version "9.0")
 	(paper "A4")
+	(title_block
+		(date "2025-09-24")
+		(company "Felix Pelster")
+	)
 	(junction
 		(at 140.97 107.95)
